Commit message: add shoulder_horn and elbow_servo links to URDF

File: rexarm_description/robots/rexarm.urdf (robot description, URDF)
Before this commit: robot goat, 4 links, 3 joints
Links:
- added link elbow_servo; visual box size=0.035 0.03 0.05
- added link shoulder_horn; visual box size=0.038 0.053 0.09
Joints:
- added joint elbow_servo_joint: type fixed, parent shoulder_horn, child elbow_servo, origin xyz=0.0 0.0 0.05 rpy=0.0 0.0 0.0
- added joint shoulder_horn_joint: type continuous, parent shoulder_servo, child shoulder_horn, origin xyz=0.0 0.0 0.029 rpy=0.0 0.0 0.0, axis 0.0 1.0 0.0
- joint shoulder_servo_joint: axis 0.0 1.0 0.0 -> 0.0 0.0 1.0

Commit message: add wrist and wrist horn

File: rexarm_description/robots/rexarm.urdf (robot description, URDF)
Before this commit: robot rexarm, 7 links, 6 joints
Links:
- added link wrist_horn; visual box size=0.034 0.049 0.05
- added link wrist_servo; visual box size=0.035 0.03 0.05
Joints:
- added joint wrist_horn_joint: type continuous, parent wrist_servo, child wrist_horn, origin xyz=0.0 0.0 0.00525 rpy=0.0 0.0 0.0, axis 0.0 1.0 0.0
- added joint wrist_servo_joint: type fixed, parent elbow_horn, child wrist_servo, origin xyz=0.0 0.0 0.079 rpy=0.0 0.0 0.0

Commit message: complete, refactor, and update rexarm URDF
* remove all visual components
* add joints and links for all servo horns

File: rexarm_description/robots/rexarm.urdf (robot description, URDF)
Before this commit: robot rexarm, 9 links, 8 joints
Links:
- removed link base_block
- removed link base_servo
- removed link elbow_horn
- removed link elbow_servo
- removed link shoulder_horn
- removed link shoulder_servo
- removed link wrist_horn
- removed link wrist_servo
- added link base_servo_link
- added link elbow_servo_link
- added link gripper_servo_link
- added link shoulder_servo_link
- added link wrist_rotate_servo_link
- added link wrist_servo_link
Joints:
- removed joint base_block_joint
- removed joint base_servo_joint
- removed joint elbow_horn_joint
- removed joint elbow_servo_joint
- removed joint shoulder_horn_joint
- removed joint shoulder_servo_joint
- removed joint wrist_horn_joint
- removed joint wrist_servo_joint
- added joint base_servo: type continuous, parent base_link, child base_servo_link, origin xyz=0.0 -0.0015 0.0715 rpy=0.0 0.0 0.0, axis 0.0 0.0 1.0
- added joint elbow_servo: type continuous, parent shoulder_servo_link, child elbow_servo_link, origin xyz=0.0 0.0 0.1 rpy=0.0 0.0 0.0, axis 0.0 1.0 0.0
- added joint gripper_servo: type continuous, parent wrist_rotate_servo_link, child gripper_servo_link, origin xyz=0.0 -0.013 0.019 rpy=0.0 0.0 0.0, axis 1.0 0.0 0.0
- added joint shoulder_servo: type continuous, parent base_servo_link, child shoulder_servo_link, origin xyz=0.0 0.0 0.045 rpy=0.0 0.0 0.0, axis 0.0 1.0 0.0
- added joint wrist_rotate_servo: type continuous, parent wrist_servo_link, child wrist_rotate_servo_link, origin xyz=0.0 -0.0125 0.08 rpy=0.0 0.0 0.0, axis 0.0 0.0 1.0
- added joint wrist_servo: type continuous, parent elbow_servo_link, child wrist_servo_link, origin xyz=0.0 0.0 0.1 rpy=0.0 0.0 0.0, axis 0.0 1.0 0.0

Commit message: add gripper_center_link to rexarm URDF
gripper_center_link corresponds to the center of the gripper, oriented
in the same way as the gripper is facing. so a neutral orientation with
all joints at zero corresponds to gripper_center_link having x facing
straight up. in other words, the x-axis of gripper_center_link is the
direction that the gripper is looking at or facing

File: rexarm_description/robots/rexarm.urdf (robot description, URDF)
Before this commit: robot rexarm, 7 links, 6 joints
Links:
- added link gripper_center_link
Joints:
- added joint gripper_center: type fixed, parent wrist_rotate_servo_link, child gripper_center_link, origin xyz=0.0 -0.005 0.07 rpy=0.0 -1.5707963267948966 0.0

Commit message: add visual tags representing mx-28, ax-12 servos

File: rexarm_description/robots/rexarm.urdf (robot description, URDF)
Before this commit: robot rexarm, 8 links, 7 joints
Links:
- link base_link: geometry visual box size=0.05 0.035 0.03
- link base_servo_link: geometry visual box size=0.035 0.03 0.05
- link elbow_servo_link: geometry visual box size=0.032 0.031 0.05
- link shoulder_servo_link: geometry visual box size=0.035 0.03 0.05
- link wrist_rotate_servo_link: geometry visual box size=0.031 0.05 0.031
- link wrist_servo_link: geometry visual box size=0.032 0.05 0.031

Commit message: add <visual> tags for fingers to rexarm URDF

File: rexarm_description/robots/rexarm.urdf (robot description, URDF)
Before this commit: robot rexarm, 8 links, 7 joints
Links:
- added link gripper_fingers_link; visual box size=0.0275 0.01 0.07
- link gripper_servo_link: geometry visual box size=0.04 0.01 0.08
Joints:
- added joint gripper_fingers: type fixed, parent wrist_rotate_servo_link, child gripper_fingers_link, origin xyz=0.0 0.01 0.07 rpy=0.0 0.0 0.0

Commit message: publish joint states with correct names+frames

File: rexarm_description/robots/rexarm.urdf (robot description, URDF)
Before this commit: robot rexarm, 9 links, 8 joints
Joints:
- added joint base: type fixed, parent arm_bundle, child base_link
